File: schematics/schematics.sch (KiCad schematic (older format))
At the start: 10 parts, among them J1 UPDI, U1 ATtiny412-SS, U2 CP2102-Module

Commit message: 図面とシフトレジスタ
Parts:
- removed D1: LED, symbol Device:LED
- removed R1: R, symbol Device:R
- added C?: 0.1u, symbol Device:C
- added D?: GREEN, symbol Device:LED
- added D?: YELLOW, symbol Device:LED
- added D?: RED, symbol Device:LED
- added R? (x3): 1K, symbol Device:R
- added U?: AE-7SEG-BOARD, symbol mamemomonga:AE-7SEG-BOARD
- added U?: 74HC595, symbol 74xx:74HC595
Connections:
- net labels added: DAC, MOSI, RX, SCK, SS
- wire segments 23 -> 63
- no-connect marks 6 -> 13
Other:
- moved on the sheet: C1, C2, J1, MES1, R2, RV1, U1, U2
