File: attiny412/schematics/schematics.kicad_sch (KiCad schematic)
At the start: 17 parts, among them J1 UPDI, U1 ATtiny412-SS, U2 CP2102-Module

Commit message: ファイル更新
Parts:
- removed C?: 10uF, symbol Device:C_Polarized
- removed MES?: 100uA, symbol Device:Ammeter_DC
- removed RV?: 50K, symbol Device:R_Potentiometer
- added C1: 10uF, symbol Device:CP
- added MES1: 100uA, symbol Device:Amperemeter_DC
- added RV1: 50K, symbol Device:R_POT
Connections:
- net DAC: now also R2.1; no longer R2.2
Other:
- moved on the sheet: C2, C?, D?, J1, R2, R?, U1, U2, U?

Commit message: 図面更新
Parts:
- removed C1: 10uF, symbol Device:CP
- removed MES1: 100uA, symbol Device:Amperemeter_DC
- removed RV1: 50K, symbol Device:R_POT
- added C1: 10uF, symbol Device:C_Polarized
- added MES1: 100uA, symbol Device:Ammeter_DC
- added RV1: 50K, symbol Device:R_Potentiometer
- gave numbers to parts that had none: 9
- renumbered R2 to R1, U2 to U1, U1 to U2
Connections:
- net +5V: now also C1.1
- net GND: now also C1.2, MES1.1 (-)
- net at R1.2: now also RV1.3
- new net: MES1.2 (+), RV1.2
